File: doc/Kicad/HomeKit_shield_ESP32_C3_FH4_1_0_0/HomeKit_shield_ESP32_C3_FH4_1_0_0.kicad_pcb (KiCad board)
At the start: 2 copper layers, 70 x 35 mm, 31 parts, among them J1 SEAN_USB_A_90, J2 SEAN_USB_A_90, J3 SEAN_USB_A_90, J5 SEAN_MTINY_I2C, J6 Conn_01x05_Socket, Q1 SEAN_MOSFET_AOD4184, Q2 SEAN_MOSFET_AOD4184, Q3 SEAN_MOSFET_AOD4184, U1 SEAN_ESP32-C3_SUPERMINI, U2 AMS1117-3.3

Commit message: Pixel
Parts:
- removed J6: Conn_01x05_Socket, Connector_PinSocket_2.00mm:PinSocket_1x05_P2.00mm_Vertical
- removed Q3: SEAN_MOSFET_AOD4184, SEAN_MOSFET:SEAN_MOSFET_AOD4184
- removed S4: SEAN_Button_4.2x3.3_SMD_V1, SEAN_Device_sym:SEAN_Button_4.2x3.3_SMD_V1
- added D4: SEAN_D, SEAN_Device_sym:SEAN_Diode_1N4007, F.Cu at (172.3, 110.6)
- added Hold_keep1: MountingHole, SEAN_MountingHole:SEAN_MountingHole_3mm_isolated, F.Cu at (148.3, 94.1)
- added J4: SEAN_Neopixel, SEAN_connect:SEAN_Neopixel, F.Cu at (160.4, 111.6)
- added J7: SEAN_USB_Type_C, SEAN_connect:SEAN_USB_Type_C, F.Cu at (180.1, 108.5)
- added K1: SEAN_Relay_G5NB, SEAN_Relay:SEAN_RELAY_HF46F, F.Cu at (124.4, 85.9)
- added Q4: S8050, Package_TO_SOT_SMD:SOT-23-3, F.Cu at (143.0, 91.8)
- added Q5: SEAN_MOSFET_bss138, SEAN_MOSFET:SEAN_MOSFET_bss138, F.Cu at (165.6, 105.1)
- added R10: 4.7K, Resistor_SMD:R_0603_1608Metric_Pad0.98x0.95mm_HandSolder, F.Cu at (210.8, 83.0)
- added R11: 10K, Resistor_SMD:R_0603_1608Metric_Pad0.98x0.95mm_HandSolder, F.Cu at (210.8, 85.5)
- added R4: 100, Resistor_SMD:R_0603_1608Metric_Pad0.98x0.95mm_HandSolder, F.Cu at (141.9, 94.5)
- added R5: 100, Resistor_SMD:R_0603_1608Metric_Pad0.98x0.95mm_HandSolder, F.Cu at (145.1, 105.8)
- added R6: 10K, Resistor_SMD:R_0603_1608Metric_Pad0.98x0.95mm_HandSolder, F.Cu at (169.9, 105.1)
- added R7: 4.7K, Resistor_SMD:R_0603_1608Metric_Pad0.98x0.95mm_HandSolder, F.Cu at (173.0, 105.8)
- added R8: 10K, Resistor_SMD:R_0603_1608Metric_Pad0.98x0.95mm_HandSolder, F.Cu at (173.0, 104.2)
- added R9: 10K, Resistor_SMD:R_0603_1608Metric_Pad0.98x0.95mm_HandSolder, F.Cu at (168.4, 105.1)
- added SEAN_Mtiny_Terminal_3.81: SEAN_Mtiny_Terminal_3.81, SEAN_Mtiny:SEAN_Mtiny_Terminal_3.81, F.Cu at (138.5, 88.1)
- added U11: ~, SEAN_mmWare:SEAN_mmWare_Rd-03, F.Cu at (149.3, 98.6)
- added U3: ~, SEAN_connect:SEAN_Hand_Solderring, B.Cu at (127.1, 112.3)
- D1, D2, D3: footprint Diode_SMD:D_0603_1608Metric_Pad1.05x0.95mm_HandSolder -> SEAN_Device_sym:SEAN_Diode_1N4007
- J3: value SEAN_USB_A_90 -> Barrel_Jack_MountingPin; footprint SEAN_connect:SEAN_USB_A_90 -> Connector_BarrelJack:BarrelJack_GCT_DCJ200-10-A_Horizontal
- R3: value 10K -> 4.7K
- moved J3 70.3 mm to (194.3, 102.0), turned to 90 degrees
- moved U8 44.3 mm to (180.7, 110.3), turned to 180 degrees
- moved U5 32.6 mm to (180.6, 106.6), turned to 180 degrees
- moved U10 22.2 mm to (120.2, 112.2)
- moved U9 22.2 mm to (117.2, 112.2)
- moved S1 16.3 mm to (148.4, 110.1)
- moved U6 16.3 mm to (148.4, 112.2)
- moved R1 14.1 mm to (141.9, 96.3), turned to 0 degrees
- moved R2 13.7 mm to (141.3, 105.8), turned to 180 degrees
- moved D2 13.4 mm to (136.0, 105.6)
- moved Q1 13.4 mm to (138.4, 101.0)
- moved Q2 13.4 mm to (138.4, 110.4)
- moved D1 13.3 mm to (136.1, 95.8)
- moved J2 11.1 mm to (124.3, 108.5)
- moved R3 10.7 mm to (138.5, 91.2)
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Connections:
- C1 pad 1: VIN -> 5v_power
- C2 pad 1: VIN -> 5v_power
- D1 pad 1: 5v -> 5v_power
- D2 pad 1: 5v -> 5v_power
- D3 pad 1: 5v -> 5v_power
- J1 pad 1: 5v -> 5v_power
- J1 pad 5: unconnected-(J1-Shield-Pad5) -> GND
- J2 pad 1: 5v -> 5v_power
- J2 pad 5: unconnected-(J2-Shield-Pad5) -> GND
- J3 pad 1: 5v -> unconnected-(J3-Pad1)
- J3 pad 3: unconnected-(J3-D+-Pad3) -> (no net)
- Q1 pad 2: GPIO_10 -> Net-(Q1-G)
- Q2 pad 2: GPIO_20 -> Net-(Q2-G)
- R1 pad 1: GPIO_10 -> Net-(Q1-G)
- R2 pad 1: GPIO_20 -> Net-(Q2-G)
- R3 pad 2: GND -> Net-(Q4-B)
- U1 pad 3.3: unconnected-(U1-3V3-Pad3.3) -> 3v3_Esp
- U1 pad 5V: 5v -> Net-(D4-K)
- U10 pad 1: GPIO_10 -> Net-(D1-A)
- U2 pad 3: VIN -> 5v_power
- U5 pad 1: GPIO_4 -> 5v_power
- U8 pad 1: GPIO_21 -> GND
- U9 pad 1: GPIO_20 -> Net-(D2-A)
Routing:
- net Net-(D4-K): track 0.00 -> 22.9 mm
- net Net-(J7-CC1): track 0.00 -> 14.6 mm
- net Net-(J7-CC2): track 0.00 -> 12.0 mm
- net 5v_power: track 0.00 -> 9.95 mm
Other:
- outline, holes or cut-outs redrawn
