File: doc/Kicad/HomeKit_shield_ESP32_C3_FH4_1_0_0/HomeKit_shield_ESP32_C3_FH4_1_0_0.kicad_sch (KiCad schematic)
At the start: 31 parts, among them J1 SEAN_USB_A_90, J2 SEAN_USB_A_90, J3 SEAN_USB_A_90, J5 SEAN_MTINY_I2C, J6 Conn_01x05_Socket, Q1 SEAN_MOSFET_AOD4184, Q2 SEAN_MOSFET_AOD4184, Q3 SEAN_MOSFET_AOD4184, U1 SEAN_ESP32-C3_SUPERMINI, U2 AMS1117-3.3

Commit message: Pixel
Parts:
- removed J3: SEAN_USB_A_90, SEAN_connect:SEAN_USB_A_90, symbol SEAN_connect:SEAN_USB_A_90
- removed J6: Conn_01x05_Socket, Connector_PinSocket_2.00mm:PinSocket_1x05_P2.00mm_Vertical, symbol Connector:Conn_01x05_Socket
- removed Q3: SEAN_MOSFET_AOD4184, SEAN_MOSFET:SEAN_MOSFET_AOD4184, symbol SEAN_MOSFET:SEAN_MOSFET_AOD4184
- removed S4: SEAN_Button_4.2x3.3_SMD_V1, SEAN_Device_sym:SEAN_Button_4.2x3.3_SMD_V1, symbol SEAN_Device_sym:SEAN_Button_4.2x3.3_SMD_V1
- added D4: SEAN_D, SEAN_Device_sym:SEAN_Diode_1N4007, symbol SEAN_Device_sym:SEAN_D
- added Hold_keep1: MountingHole, SEAN_MountingHole:SEAN_MountingHole_3mm_isolated, symbol Mechanical:MountingHole
- added J4: SEAN_Neopixel, SEAN_connect:SEAN_Neopixel, symbol SEAN_connect:SEAN_Neopixel
- added J7: SEAN_USB_Type_C, SEAN_connect:SEAN_USB_Type_C, symbol SEAN_connect:SEAN_USB_Type_C
- added K1: SEAN_Relay_G5NB, SEAN_Relay:SEAN_RELAY_HF46F, symbol SEAN_Relay:SEAN_Relay_G5NB
- added Q4: S8050, Package_TO_SOT_SMD:SOT-23-3, symbol Transistor_BJT:S8050
- added Q5: SEAN_MOSFET_bss138, SEAN_MOSFET:SEAN_MOSFET_bss138, symbol SEAN_MOSFET:SEAN_MOSFET_bss138
- added R10, R7: 4.7K, Resistor_SMD:R_0603_1608Metric_Pad0.98x0.95mm_HandSolder, symbol SEAN_Device_sym:SEAN_R
- added R11, R6, R8, R9: 10K, Resistor_SMD:R_0603_1608Metric_Pad0.98x0.95mm_HandSolder, symbol SEAN_Device_sym:SEAN_R
- added R4, R5: 100, Resistor_SMD:R_0603_1608Metric_Pad0.98x0.95mm_HandSolder, symbol SEAN_Device_sym:SEAN_R
- added SEAN_Mtiny_Terminal_3.81: SEAN_Mtiny_Terminal_3.81, SEAN_Mtiny:SEAN_Mtiny_Terminal_3.81, symbol SEAN_Mtiny:SEAN_Mtiny_Terminal_3.81
- added U11: ~, SEAN_mmWare:SEAN_mmWare_Rd-03, symbol SEAN_mmWare:SEAN_mmWare_Rd-03
- added U3: ~, SEAN_connect:SEAN_Hand_Solderring, symbol SEAN_connect:SEAN_Hand_Solderring
- D1, D2, D3: footprint Diode_SMD:D_0603_1608Metric_Pad1.05x0.95mm_HandSolder -> SEAN_Device_sym:SEAN_Diode_1N4007
- R3: value 10K -> 4.7K
Connections:
- net 3v3: now also U11.5 (3v3)
- net 5v: no longer D1.1 (K), D2.1 (K), D3.1 (K), J1.1 (VBUS), J2.1 (VBUS), U1.5V
- net GND: now also J1.5 (Shield), J2.5 (Shield), U8.1 (Hand_Soldering), J4.1 (GND), J7.A1 (GND), J7.A12 (GND), J7.B1 (GND), J7.B12 (GND), J7.S1 (SHIELD), Q4.1 (E), R10.1, R7.1, U11.4 (GND), U3.1 (Hand_Soldering); no longer R3.2
- net GPIO_10: now also R4.2; no longer Q1.2 (G), R1.1, U10.1 (Hand_Soldering)
- net GPIO_2: now also Q5.3 (S), R6.2
- net GPIO_20: now also R5.2; no longer Q2.2 (G), R2.1, U9.1 (Hand_Soldering)
- net GPIO_21: no longer U8.1 (Hand_Soldering)
- net GPIO_4: no longer U5.1 (Hand_Soldering)
- net GPIO_5-SDA: now also R8.2
- net GPIO_6-SCL: now also R11.2
- net GPIO_7: now also U11.1 (TX1)
- net at D1.2 (A), J1.4 (GND), Q1.1 (D): now also U10.1 (Hand_Soldering)
- net at D2.2 (A), J2.4 (GND), Q2.1 (D): now also U9.1 (Hand_Soldering)
- net at D3.2 (A): now also K1.2, Q4.3 (C)
- net 3v3_Esp: now reaches U1.3.3 (3V3)
- net 3v3_Esp: now also Q5.2 (G), R11.1, R6.1, R8.1
- net VIN renamed 5v_power
- net 5v_power: now also D1.1 (K), D2.1 (K), D3.1 (K), J1.1 (VBUS), J2.1 (VBUS), U5.1 (Hand_Soldering), D4.1 (K), J4.3 (SDA), J7.A4 (VBUS), J7.A9 (VBUS), J7.B4 (VBUS), J7.B9 (VBUS), K1.1, R9.2
- new net: J4.2 (5V), Q5.1 (D), R9.1
- new net: Q4.2 (B), R3.2
- new net: Q2.2 (G), R2.1, R5.1
- new net: Q1.2 (G), R1.1, R4.1
- new net: J7.A5 (CC1), R7.2
- new net: J7.B5 (CC2), R10.2
- new net: D4.2 (A), U1.5V
- new net: K1.3, SEAN_Mtiny_Terminal_3.81.1 (Pin_1)
- new net: K1.4, SEAN_Mtiny_Terminal_3.81.2 (Pin_2)
Other:
- note added: "ESP32-C3 Super Mini"
- note added: "Hold"
- note added: "Neopixel"
- note added: "Power 3v3"
- note added: "Relay"
- note added: "USB control"
- note added: "Usb_C_power"
- moved on the sheet: D1, D2, J1, J2, Q1, Q2, S1, S2, S3, U1

Commit message: auto AP Wifi
Parts:
- removed D1, D2, D3, D4: SEAN_D, SEAN_Device_sym:SEAN_Diode_1N4007, symbol SEAN_Device_sym:SEAN_D
- removed Hold_keep1: MountingHole, SEAN_MountingHole:SEAN_MountingHole_3mm_isolated, symbol Mechanical:MountingHole
- removed J1, J2: SEAN_USB_A_90, SEAN_connect:SEAN_USB_A_90, symbol SEAN_connect:SEAN_USB_A_90
- removed J4: SEAN_Neopixel, SEAN_connect:SEAN_Neopixel, symbol SEAN_connect:SEAN_Neopixel
- removed J5: SEAN_MTINY_I2C, SEAN_Mtiny:SEAN_Mtiny_I2C, symbol SEAN_Mtiny:SEAN_MTINY_I2C
- removed J7: SEAN_USB_Type_C, SEAN_connect:SEAN_USB_Type_C, symbol SEAN_connect:SEAN_USB_Type_C
- removed K1: SEAN_Relay_G5NB, SEAN_Relay:SEAN_RELAY_HF46F, symbol SEAN_Relay:SEAN_Relay_G5NB
- removed Q1, Q2: SEAN_MOSFET_AOD4184, SEAN_MOSFET:SEAN_MOSFET_AOD4184, symbol SEAN_MOSFET:SEAN_MOSFET_AOD4184
- removed Q4: S8050, Package_TO_SOT_SMD:SOT-23-3, symbol Transistor_BJT:S8050
- removed Q5: SEAN_MOSFET_bss138, SEAN_MOSFET:SEAN_MOSFET_bss138, symbol SEAN_MOSFET:SEAN_MOSFET_bss138
- removed R1, R11, R2, R6, R8, R9: 10K, Resistor_SMD:R_0603_1608Metric_Pad0.98x0.95mm_HandSolder, symbol SEAN_Device_sym:SEAN_R
- removed R10, R3, R7: 4.7K, Resistor_SMD:R_0603_1608Metric_Pad0.98x0.95mm_HandSolder, symbol SEAN_Device_sym:SEAN_R
- removed R4, R5: 100, Resistor_SMD:R_0603_1608Metric_Pad0.98x0.95mm_HandSolder, symbol SEAN_Device_sym:SEAN_R
- removed SEAN_Mtiny_Terminal_3.81: SEAN_Mtiny_Terminal_3.81, SEAN_Mtiny:SEAN_Mtiny_Terminal_3.81, symbol SEAN_Mtiny:SEAN_Mtiny_Terminal_3.81
- removed U10, U3, U4, U5, U6, U7, U8, U9: ~, SEAN_connect:SEAN_Hand_Solderring, symbol SEAN_connect:SEAN_Hand_Solderring
- added C5: 100nF, Capacitor_SMD:C_0603_1608Metric_Pad1.08x0.95mm_HandSolder, symbol SEAN_Device_sym:SEAN_C
- added J1: Conn_01x03_Socket, symbol Connector:Conn_01x03_Socket
- added S4: SEAN_Button_4.2x3.3_SMD_V1, SEAN_Device_sym:SEAN_Button_4.2x3.3_SMD_V1, symbol SEAN_Device_sym:SEAN_Button_4.2x3.3_SMD_V1
Connections:
- net 3v3: now also C5.2
- net 5v_power: now also U1.5V
- net GND: now also C5.1, S4.1, S4.2
- net GPIO_0: now also S4.3, S4.4; no longer S1.3, S1.4
- net GPIO_1: now also U11.1 (TX1); no longer S2.3, S2.4
- net GPIO_10: now also S1.3, S1.4
- net GPIO_3: now also J1.3 (Pin_3); no longer S3.3, S3.4
- net GPIO_4: now also J1.2 (Pin_2)
- net GPIO_7: now also S2.3, S2.4; no longer U11.1 (TX1)
- net GPIO_5-SDA renamed GPIO_5
- net GPIO_5: now also J1.1 (Pin_1)
- net GPIO_6-SCL renamed GPIO_6
- net GPIO_6: now also S3.3, S3.4
Other:
- note added: "RD-03"
- note removed: "Hold"
- note removed: "Neopixel"
- note removed: "Relay"
- note removed: "USB control"
- note removed: "Usb_C_power"
- company: (none) -> MakerLab.vn
- moved on the sheet: U1, U11
